File: Schematic/BMS.sch (KiCad schematic (older format))
At the start: 0 parts

Commit message: Add files via upload
Parts:
- added CAN1: Conn_01x02, symbol Connector_Generic:Conn_01x02
- added Debug1: Conn_01x06, symbol Connector_Generic:Conn_01x06
- added J?: Charging_Connector, symbol Connector_Generic:Conn_01x02
- added J?: Load_Connector, symbol Connector_Generic:Conn_01x02
- added J?: Battery_Balancing_Con, symbol Connector_Generic:Conn_01x07
Connections:
- net labels added: CANH, CANL, GND, SWCLK, SWDIO, USART_RX, USART_TX, V_3.3
- wire segments 0 -> 54
Other:
- note removed: "Cell Protection and Balancing"
- note removed: "Controller\n\n"
- note removed: "DC to DC Converter\n"
- note removed: "USB Power Delivery"

Commit message: Add files via upload
Parts:
- removed CAN1: Conn_01x02, symbol Connector_Generic:Conn_01x02
- removed Debug1: Conn_01x06, symbol Connector_Generic:Conn_01x06
- removed J?: Load_Connector, symbol Connector_Generic:Conn_01x02
- added D?: D, symbol Device:D
- added F?: Fuse, symbol Device:Fuse
- added J?: Battery_Connector, symbol Connector_Generic:Conn_01x02
- added J?: Load_Connector, symbol Connector_Generic:Conn_01x02
- added Q?: CSD18543Q3AT, ASSETS:CSD18543Q3AT, symbol Regular_Use:CSD18543Q3AT
Connections:
- net labels added: IM_SWITCH
- net labels removed: CANH, CANL, SWCLK, SWDIO, USART_RX, USART_TX, V_3.3
- wire segments 54 -> 111
Other:
- moved on the sheet: J?
