File: Schematic/Cell_Balancing.sch (KiCad schematic (older format))
At the start: 27 parts

Commit message: Add files via upload
Changed lines of the file:
@@
 Wire Notes Line
 	550  600  550  3600
+Wire Wire Line
+	1500 8850 1600 8850
+Text HLabel 1600 8850 2    50   Input Italic 0
+V_3.3
+Text GLabel 1500 8850 0    50   Input Italic 0
+V_3.3
 $EndSCHEMATC
