File: Schematic/controller.sch (KiCad schematic (older format))
At the start: 1 part

Commit message: Add files via upload
Changed lines of the file:
@@
 $Descr A4 8268 11693 portrait
 encoding utf-8
-Sheet 4 6
+Sheet 4 7
 Title ""
 Date ""
@@
 	1    0    0    -1
 $EndComp
+Text GLabel 6600 4500 0    50   Input Italic 0
+IM_SWITCH
+Text GLabel 6600 4650 0    50   Input Italic 0
+D+
+Text GLabel 6600 4800 0    50   Input Italic 0
+D-
+Text GLabel 6600 4950 0    50   Input Italic 0
+V_SENSE
+Text GLabel 6600 5250 0    50   Input Italic 0
+SCL
+Text GLabel 6600 5400 0    50   Input Italic 0
+SDA
+Text GLabel 6600 5550 0    50   Input Italic 0
+nALERT
+Text GLabel 6600 5700 0    50   Input Italic 0
+MOSI
+Text GLabel 6600 5850 0    50   Input Italic 0
+TX_EN
+Text GLabel 6600 6000 0    50   Input Italic 0
+SCLK
+Text GLabel 6600 6150 0    50   Input Italic 0
+NSS
+Text GLabel 6600 6300 0    50   Input Italic 0
+MISO
+Text GLabel 6600 6450 0    50   Input Italic 0
+V_3.3
+Text HLabel 6700 4500 2    50   Input Italic 0
+IM_SWITCH
+Text HLabel 6700 4650 2    50   Input Italic 0
+D+
+Text HLabel 6700 4800 2    50   Input Italic 0
+D-
+Text HLabel 6700 4950 2    50   Input Italic 0
+V_SENSE
+Text HLabel 6700 5250 2    50   Input Italic 0
+SCL
+Text HLabel 6700 5400 2    50   Input Italic 0
+SDA
+Text HLabel 6700 5550 2    50   Input Italic 0
+nALERT
+Text HLabel 6700 5700 2    50   Input Italic 0
+MOSI
+Text HLabel 6700 5850 2    50   Input Italic 0
+TX_EN
+Text HLabel 6700 6000 2    50   Input Italic 0
+SCLK
+Text HLabel 6700 6150 2    50   Input Italic 0
+NSS
+Text HLabel 6700 6300 2    50   Input Italic 0
+MISO
+Text HLabel 6700 6450 2    50   Input Italic 0
+V_3.3
+Wire Wire Line
+	6600 4500 6700 4500
+Wire Wire Line
+	6600 4650 6700 4650
+Wire Wire Line
+	6600 4800 6700 4800
+Wire Wire Line
+	6600 4950 6700 4950
+Wire Wire Line
+	6600 5250 6700 5250
+Wire Wire Line
+	6600 5400 6700 5400
+Wire Wire Line
+	6600 5550 6700 5550
+Wire Wire Line
+	6600 5700 6700 5700
+Wire Wire Line
+	6600 5850 6700 5850
+Wire Wire Line
+	6600 6000 6700 6000
+Wire Wire Line
+	6600 6150 6700 6150
+Wire Wire Line
+	6600 6300 6700 6300
+Wire Wire Line
+	6600 6450 6700 6450
 $EndSCHEMATC
