File: Schematic/prot_bal.sch (KiCad schematic (older format))
At the start: 58 parts

Commit message: Add files via upload
Parts:
- removed BT? (x5): Battery_Cell, symbol Device:Battery_Cell
- removed C? (x6): C_Small, symbol Device:C_Small
- removed C? (x6): 1U, symbol Device:C_Small
- removed IC? (x6): BQ29707DSER, ASSETS:SON50P150X150X80-6N, symbol Regular_Use:BQ29707DSER
- removed IC?: BQ7692006PWR, ASSETS:SOP65P640X120-20N, symbol Regular_Use:BQ7692006PWR
- removed J?: Conn_01x05, symbol Connector_Generic:Conn_01x05
- removed Q? (x14): DMG3402L, Package_TO_SOT_SMD:SOT-23, symbol Transistor_FET:DMG3402L
- removed R? (x12): R_Small, symbol Device:R_Small
- removed R? (x6): 1K, symbol Device:R_Small
- removed U?: BQ76PL536PAP, ASSETS:QFP50P1200X1200X120-65N, symbol Regular_Use:BQ76PL536PAP
- added C? (x2): 10UF, symbol Device:C_Small
- added C? (x4): 2.2UF, symbol Device:C_Small
- added C? (x2): 0.047UF, symbol Device:C_Small
- added C? (x3): 1UF, symbol Device:C_Small
- added D?: LED, symbol Device:LED
- added J?: Conn_01x07, symbol Connector_Generic:Conn_01x07
- added J?: Conn_01x02, symbol Connector_Generic:Conn_01x02
- added Q?: DMG3402L, Package_TO_SOT_SMD:SOT-23, symbol Transistor_FET:DMG3402L
- added R? (x4): R_Small, symbol Device:R_Small
- added R?: 2.7K, symbol Device:R_Small
- added R?: 100, symbol Device:R_Small
- added R?: 100K, symbol Device:R_Small
- added R? (x2): 0, symbol Device:R_Small
- added TH? (x2): NTC0603, symbol Device:Thermistor_NTC
- added U?: BQ76PL536PAP, ASSETS:QFP50P1200X1200X120-65N, symbol Regular_Use:BQ76PL536PAP
Connections:
- net labels added: ALERT_H, AUX, CONV_H, CS_H, DRDY_H, FAULT_H, SCLK_H, SDI_H, SDO_H
- net labels removed: LDOD2, REG50
- wire segments 227 -> 204
- no-connect marks 0 -> 16
Other:
- note removed: "V_S 22 DRDY_S 23 ALERT_S 24 FAULT_S\n25 VSS2\n26 SCLK_S 27 SDO_S 28 SDI_S 29 CS_S"
