File: Schematic/DC_DC_Converter.sch (KiCad schematic (older format))
At the start: 37 parts

Commit message: Add files via upload
Parts:
- added F?: Fuse, symbol Device:Fuse
- added U?: LM34936_NEW, ASSETS:QFN50P400X500X100-29N-D, symbol Regular_Use:LM34936_NEW
- gave numbers to parts that had none: 4
Connections:
- net BPPT1 is gone; now on net BOOT1: IC?.23 (BOOT1)
- net BOOT1: now also U?.23 (BOOT1)
- net BOOT2: now also U?.17 (BOOT2)
- net EN_UVLO: now also U?.26 (VISNS)
- net FB: now also U?.8 (FB)
- net HDRV1: now also U?.24 (HDRV1); no longer Q3.1 (G)
- net HDRV2: now also Q3.1 (G), U?.16 (HDRV2)
- net LDRV1: now also U?.22 (LDRV1); no longer Q4.1 (G)
- net LDRV2: now also Q4.1 (G)
- net PWR_IN: now also C?.1, C?.1, D?.2 (A), Q1.3 (D), R?.1, R?.1; no longer C?.1, C?.1, C?.1, C?.1, IC?.9 (VOSNS), Q3.3 (D), R?.1
- net SW1: now also U?.25 (SW1)
- net SW2: now also U?.15 (SW2)
- net VIN: now also U?.27 (VIN)
- net VISNS: now also U?.26 (VISNS)
- net at C?.1, R?.1: now also U?.12 (CSG); no longer IC?.12 (CSG)
- net at C?.2, R?.2: now also U?.13 (CS); no longer IC?.13 (CS)
- net VSONS renamed VOSNS
- net VOSNS: now also C?.1, C?.1, C?.1, C?.1, IC?.9 (VOSNS), Q3.3 (D), R?.1, F?.2, U?.21 (BIAS), U?.9 (VOSNS)
- new net PWR_OUT: F?.1
Other:
- moved on the sheet: C?, D?, IC?, L?, Q?, R?
