File: Schematic/_autosave-Protection.sch (KiCad schematic (older format))
At the start: 45 parts, among them IC3 BQ7693003DBTR, Q10 DMG3402L, Q6 DMG2301L, Q7 SISA72DN-T1-GE3, Q8 SISA72DN-T1-GE3, Q9 DMG3402L

Commit message: Add files via upload
Changed lines of the file:
@@
 Wire Wire Line
 	2250 9950 2250 10050
-Text GLabel 2800 6850 2    50   BiDi Italic 0
+Text GLabel 2800 6850 2    50   Input Italic 0
 VC10
-Text GLabel 2800 7300 2    50   BiDi Italic 0
+Text GLabel 2800 7300 2    50   Input Italic 0
 VC7
-Text GLabel 2800 7750 2    50   BiDi Italic 0
+Text GLabel 2800 7750 2    50   Input Italic 0
 VC6
-Text GLabel 2800 8350 2    50   BiDi Italic 0
+Text GLabel 2800 8350 2    50   Input Italic 0
 VC5B
 Wire Wire Line
@@
 Connection ~ 2250 6850
 Connection ~ 2250 8800
-Text GLabel 2800 8800 2    50   BiDi Italic 0
+Text GLabel 2800 8800 2    50   Input Italic 0
 VC5
 Wire Wire Line
 	2250 8800 2800 8800
-Text GLabel 2800 9200 2    50   BiDi Italic 0
+Text GLabel 2800 9200 2    50   Input Italic 0
 VC2
 Wire Wire Line
 	2250 9200 2800 9200
-Text GLabel 2800 9700 2    50   BiDi Italic 0
+Text GLabel 2800 9700 2    50   Input Italic 0
 VC1
 Wire Wire Line
@@
 Wire Wire Line
 	2250 10050 2250 10100
-Text GLabel 2850 10500 2    50   BiDi Italic 0
+Text GLabel 2850 10500 2    50   Input Italic 0
 VC0
 Wire Wire Line
@@
 Wire Wire Line
 	2900 1100 2900 1500
+Text GLabel 9100 8500 0    50   BiDi Italic 0
+ALERT
+Text GLabel 8850 8650 2    50   BiDi Italic 0
+SCL
+Text GLabel 8850 8750 2    50   BiDi Italic 0
+SDA
 $EndSCHEMATC
