File: Schematic/Bal_Fet.sch (KiCad schematic (older format))
At the start: 54 parts

Commit message: Add files via upload
Connections:
- net VC0 is gone; now on net GND: C?.2, D?.2 (A), D?.2 (A), Q?.2 (S), R?.1
Changed lines of the file:
@@
 $Descr A4 8268 11693 portrait
 encoding utf-8
-Sheet 7 6
+Sheet 6 6
 Title ""
 Date ""
@@
 $EndComp
 Wire Wire Line
-	4550 9350 5950 9350
+	4550 9350 5550 9350
+Wire Wire Line
+	5550 9350 5550 9650
+Connection ~ 5550 9350
+Wire Wire Line
+	5550 9350 5950 9350
+$Comp
+L power:GND #PWR?
+U 1 1 5F9DC089
+P 5550 9650
+F 0 "#PWR?" H 5550 9400 50  0001 C CNN
+F 1 "GND" H 5555 9477 50  0000 C CNN
+F 2 "" H 5550 9650 50  0001 C CNN
+F 3 "" H 5550 9650 50  0001 C CNN
+	1    5550 9650
+	1    0    0    -1
+$EndComp
 $EndSCHEMATC
